Commit message: Lots of changes to make gz/rviz/amcl work together

File: ros2/ros_ws/src/tb4_description/urdf/icreate/common_properties.urdf.xacro (robot description, xacro)
@@ -49,6 +49,5 @@
       <visualize>${visualize}</visualize>
       <always_on>true</always_on>
-      <!-- <gz_frame_id>${namespace}/${sensor_name}_link</gz_frame_id> -->
-      <gz_frame_id>${sensor_name}_link</gz_frame_id>
+      <gz_frame_id>${namespace}/${sensor_name}_link</gz_frame_id>
       <topic>${namespace}/scan</topic>
       <lidar>

File: ros2/ros_ws/src/tb4_description/urdf/icreate/create3.urdf.xacro (robot description, xacro)
@@ -6,8 +6,6 @@
   <xacro:include filename="$(find tb4_description)/urdf/icreate/sensors/imu.urdf.xacro" />
   <xacro:include filename="$(find tb4_description)/urdf/icreate/wheel.urdf.xacro" />
-  <!-- Gazebo version -->
-  <xacro:arg name="gazebo"                       default="gazebo" />
-  <!-- Namespace -->
-  <xacro:arg name="namespace"                    default=""/>
+  <!-- <xacro:property name="namespace" value="$(arg namespace)" /> -->
+  <!-- <xacro:property name="clean_namespace" value="${namespace.replace('/', '')}" /> -->
   <!-- Mechanical properties -->
   <xacro:property name="body_z_offset"           value="${-2.5*cm2m}" />
@@ -52,5 +50,5 @@
   <xacro:bumper
       gazebo="$(arg gazebo)"
-      namespace="$(arg namespace)"
+      namespace="${clean_namespace}"
       visual_mesh="package://tb4_description/meshes/bumper_visual.dae"
       collision_mesh="package://tb4_description/meshes/bumper_collision.dae">
@@ -75,5 +73,5 @@
   </xacro:caster>
   <!-- IMU -->
-  <xacro:imu_sensor gazebo="$(arg gazebo)" namespace="$(arg namespace)">
+  <xacro:imu_sensor gazebo="$(arg gazebo)" namespace="${clean_namespace}">
     <origin xyz="0.050613 0.043673 ${0.0202 + base_link_z_offset}"/>
   </xacro:imu_sensor>
@@ -94,9 +92,9 @@
         <max_angular_velocity>2.0</max_angular_velocity>
         <min_angular_velocity>-2.0</min_angular_velocity>
-      <topic>$(arg namespace)/cmd_vel</topic>
-        <odom_topic>$(arg namespace)/odom</odom_topic>
-        <tf_topic>$(arg namespace)/tf</tf_topic>
-        <frame_id>odom</frame_id>
-        <child_frame_id>base_link</child_frame_id>
+      <topic>${clean_namespace}/cmd_vel</topic>
+        <odom_topic>${clean_namespace}/odom</odom_topic>
+        <tf_topic>${clean_namespace}/tf</tf_topic>
+        <frame_id>${clean_namespace}/odom</frame_id>
+        <child_frame_id>${clean_namespace}/base_link</child_frame_id>
         <odom_publish_frequency>10</odom_publish_frequency>
       </plugin>
@@ -106,5 +104,5 @@
         <joint_name>left_wheel_joint</joint_name>
         <joint_name>right_wheel_joint</joint_name>
-        <topic>$(arg namespace)/joint_states</topic>
+        <topic>${clean_namespace}/joint_states</topic>
         <update_rate>10</update_rate>
       </plugin>

File: ros2/ros_ws/src/tb4_description/urdf/sensors/oakd.urdf.xacro (robot description, xacro)
@@ -115,5 +115,5 @@
       <update_rate>10</update_rate>
       <visualize>true</visualize>
-        <topic>$(arg namespace)/rgbd_camera</topic>
+        <topic>${clean_namespace}/rgbd_camera</topic>
     </sensor>
     <xacro:material_darkgray/>

File: ros2/ros_ws/src/tb4_description/urdf/standard/turtlebot4.urdf.xacro (robot description, xacro)
@@ -1,4 +1,10 @@
 <?xml version="1.0" ?>
 <robot name="turtlebot4" xmlns:xacro="http://ros.org/wiki/xacro">
+  <!-- Gazebo version -->
+  <xacro:arg name="gazebo"                       default="harmonic" />
+  <!-- Namespace -->
+  <xacro:arg name="namespace"                    default=""/>
+  <xacro:property name="namespace" value="$(arg namespace)" />
+  <xacro:property name="clean_namespace" value="${namespace.replace('/', '')}" />
   <!-- Base create3 model -->
   <xacro:include filename="$(find tb4_description)/urdf/icreate/create3.urdf.xacro" />
@@ -110,5 +116,5 @@
   </xacro:tower_sensor_plate>
   <!-- Turtlebot4 sensor definitions -->
-  <xacro:rplidar name="rplidar" namespace="$(arg namespace)" parent_link="shell_link" gazebo="$(arg gazebo)">
+  <xacro:rplidar name="rplidar" namespace="${clean_namespace}" parent_link="shell_link" gazebo="$(arg gazebo)">
     <origin xyz="${rplidar_x_offset} ${rplidar_y_offset} ${rplidar_z_offset}"
             rpy="0 0 0"/>
