Commit message: Remove IMU

File: ros2/ros_ws/src/tb4_description/urdf/icreate/create3.urdf.xacro (robot description, xacro)
@@ -4,5 +4,5 @@
   <xacro:include filename="$(find tb4_description)/urdf/icreate/caster.urdf.xacro" />
   <xacro:include filename="$(find tb4_description)/urdf/icreate/common_properties.urdf.xacro"/>
-  <xacro:include filename="$(find tb4_description)/urdf/icreate/sensors/imu.urdf.xacro" />
+  <!-- <xacro:include filename="$(find tb4_description)/urdf/icreate/sensors/imu.urdf.xacro" /> -->
   <xacro:include filename="$(find tb4_description)/urdf/icreate/wheel.urdf.xacro" />
   <!-- <xacro:property name="namespace" value="$(arg namespace)" /> -->
@@ -73,7 +73,7 @@
   </xacro:caster>
   <!-- IMU -->
-  <xacro:imu_sensor gazebo="$(arg gazebo)" namespace="${clean_namespace}">
-    <origin xyz="0.050613 0.043673 ${0.0202 + base_link_z_offset}"/>
-  </xacro:imu_sensor>
+  <!-- <xacro:imu_sensor gazebo="$(arg gazebo)" namespace="${clean_namespace}"> -->
+  <!--   <origin xyz="0.050613 0.043673 ${0.0202 + base_link_z_offset}"/> -->
+  <!-- </xacro:imu_sensor> -->
   <gazebo>
       <plugin

File: ros2/ros_ws/src/tb4_description/urdf/sensors/oakd.urdf.xacro (robot description, xacro)
@@ -89,12 +89,12 @@
   </joint>
   <!-- IMU -->
-  <link name="${name}_imu_frame">
-    <xacro:inertial_dummy/>
-  </link>
-  <joint name="${name}_imu_joint" type="fixed">
-      <parent link="${base_frame}"/>
-      <child link="${name}_imu_frame"/>
-      <origin xyz="0 0 0" rpy="-${M_PI/2} 0 -${M_PI/2}" />
-  </joint>
+  <!-- <link name="${name}_imu_frame"> -->
+  <!--   <xacro:inertial_dummy/> -->
+  <!-- </link> -->
+  <!-- <joint name="${name}_imu_joint" type="fixed"> -->
+  <!--     <parent link="${base_frame}"/> -->
+  <!--     <child link="${name}_imu_frame"/> -->
+  <!--     <origin xyz="0 0 0" rpy="-${M_PI/2} 0 -${M_PI/2}" /> -->
+  <!-- </joint> -->
   <!-- Gazebo links and joints -->
   <gazebo reference="${name}_rgb_camera_frame">
@@ -140,7 +140,7 @@
     <preserveFixedJoint>true</preserveFixedJoint>
   </gazebo>
-  <gazebo reference="${name}_imu_joint">
-    <preserveFixedJoint>true</preserveFixedJoint>
-  </gazebo>
+  <!-- <gazebo reference="${name}_imu_joint"> -->
+  <!--   <preserveFixedJoint>true</preserveFixedJoint> -->
+  <!-- </gazebo> -->
 </xacro:macro>
 </robot>
